File: generator.kicad_sch.kicad_sch (KiCad schematic)
At the start: 5 parts, among them U3 NE555D

Commit message: values corrected, 40KHz generator modified
Parts:
- C17: value C_Small -> 0.47n
- C18: value C_Small -> 0.01u
- R26: value R_Small -> 560K
- R27: value R_Small -> 39K
Connections:
- net 40KHz: now also R27.1
- net at C17.1, R27.2, U3.2 (TR)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: now also R26.2
- now unconnected: U3.7 (DIS)
Other:
- moved on the sheet: R27
Changed lines of the file:
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@@
   (junction (at 146.05 101.6) (diameter 0) (color 0 0 0 0)
-  )
-  (junction (at 149.86 91.44) (diameter 0) (color 0 0 0 0)
   )
   (junction (at 121.92 82.55) (diameter 0) (color 0 0 0 0)
   )
+  (junction (at 149.86 101.6) (diameter 0) (color 0 0 0 0)
+  )
+  (junction (at 140.97 101.6) (diameter 0) (color 0 0 0 0)
+  )
   (junction (at 121.92 110.49) (diameter 0) (color 0 0 0 0)
   )
-  (junction (at 149.86 101.6) (diameter 0) (color 0 0 0 0)
+  (junction (at 135.89 91.44) (diameter 0) (color 0 0 0 0)
+  )
+  (wire (pts (xy 135.89 91.44) (xy 137.16 91.44))
+    (stroke (width 0) (type default) (color 0 0 0 0))
   )
   (wire (pts (xy 104.14 96.52) (xy 109.22 96.52))
@@
     (stroke (width 0) (type default) (color 0 0 0 0))
   )
-  (wire (pts (xy 102.87 82.55) (xy 121.92 82.55))
+  (wire (pts (xy 140.97 95.25) (xy 140.97 93.98))
     (stroke (width 0) (type default) (color 0 0 0 0))
   )
-  (wire (pts (xy 134.62 96.52) (xy 146.05 96.52))
+  (wire (pts (xy 149.86 88.9) (xy 149.86 101.6))
     (stroke (width 0) (type default) (color 0 0 0 0))
   )
-  (wire (pts (xy 149.86 101.6) (xy 149.86 99.06))
+  (wire (pts (xy 102.87 82.55) (xy 121.92 82.55))
     (stroke (width 0) (type default) (color 0 0 0 0))
   )
@@
     (stroke (width 0) (type default) (color 0 0 0 0))
   )
-  (wire (pts (xy 149.86 91.44) (xy 149.86 93.98))
+  (wire (pts (xy 140.97 100.33) (xy 140.97 101.6))
     (stroke (width 0) (type default) (color 0 0 0 0))
   )
   (wire (pts (xy 149.86 83.82) (xy 149.86 82.55))
-    (stroke (width 0) (type default) (color 0 0 0 0))
-  )
-  (wire (pts (xy 146.05 96.52) (xy 146.05 91.44))
     (stroke (width 0) (type default) (color 0 0 0 0))
   )
@@
     (stroke (width 0) (type default) (color 0 0 0 0))
   )
+  (wire (pts (xy 135.89 93.98) (xy 135.89 91.44))
+    (stroke (width 0) (type default) (color 0 0 0 0))
+  )
   (wire (pts (xy 106.68 91.44) (xy 106.68 109.22))
+    (stroke (width 0) (type default) (color 0 0 0 0))
+  )
+  (wire (pts (xy 140.97 101.6) (xy 146.05 101.6))
+    (stroke (width 0) (type default) (color 0 0 0 0))
+  )
+  (wire (pts (xy 135.89 93.98) (xy 140.97 93.98))
     (stroke (width 0) (type default) (color 0 0 0 0))
   )
@@
     (stroke (width 0) (type default) (color 0 0 0 0))
   )
-  (wire (pts (xy 134.62 101.6) (xy 146.05 101.6))
+  (wire (pts (xy 134.62 101.6) (xy 140.97 101.6))
     (stroke (width 0) (type default) (color 0 0 0 0))
   )
-  (wire (pts (xy 134.62 91.44) (xy 137.16 91.44))
-    (stroke (width 0) (type default) (color 0 0 0 0))
-  )
-  (wire (pts (xy 149.86 91.44) (xy 149.86 88.9))
-    (stroke (width 0) (type default) (color 0 0 0 0))
-  )
-  (wire (pts (xy 146.05 91.44) (xy 149.86 91.44))
+  (wire (pts (xy 134.62 91.44) (xy 135.89 91.44))
     (stroke (width 0) (type default) (color 0 0 0 0))
   )
@@
       (effects (font (size 1.27 1.27)) (justify left))
     )
-    (property "Value" "C_Small" (id 1) (at 152.4 106.6862 0)
+    (property "Value" "0.47n" (id 1) (at 152.4 106.6862 0)
       (effects (font (size 1.27 1.27)) (justify left))
     )
@@
       (effects (font (size 1.27 1.27)) (justify left))
     )
-    (property "Value" "C_Small" (id 1) (at 93.98 107.95 0)
+    (property "Value" "0.01u" (id 1) (at 96.52 107.95 0)
       (effects (font (size 1.27 1.27)) (justify left))
     )
@@
       (effects (font (size 1.27 1.27)) (justify left))
     )
-    (property "Value" "R_Small" (id 1) (at 152.4 87.6299 0)
+    (property "Value" "560K" (id 1) (at 152.4 87.6299 0)
       (effects (font (size 1.27 1.27)) (justify left))
     )
@@
     (pin "2")
   )
-  (symbol (lib_id "Device:R_Small") (at 149.86 96.52 0) (unit 1)
+  (symbol (lib_id "Device:R_Small") (at 140.97 97.79 0) (unit 1)
     (in_bom yes) (on_board yes) (fields_autoplaced)
-    (property "Reference" "R27" (id 0) (at 152.4 95.2499 0)
+    (property "Reference" "R27" (id 0) (at 143.51 96.5199 0)
       (effects (font (size 1.27 1.27)) (justify left))
     )
-    (property "Value" "R_Small" (id 1) (at 152.4 97.7899 0)
+    (property "Value" "39K" (id 1) (at 143.51 99.0599 0)
       (effects (font (size 1.27 1.27)) (justify left))
     )
-    (property "Footprint" "Resistor_SMD:R_0603_1608Metric" (id 2) (at 149.86 96.52 0)
+    (property "Footprint" "Resistor_SMD:R_0603_1608Metric" (id 2) (at 140.97 97.79 0)
       (effects (font (size 1.27 1.27)) hide)
     )
-    (property "Datasheet" "~" (id 3) (at 149.86 96.52 0)
+    (property "Datasheet" "~" (id 3) (at 140.97 97.79 0)
       (effects (font (size 1.27 1.27)) hide)
     )
